File: eagle/logic3.1.sch (EAGLE design)
At the start: 76 parts, among them IC1 MCP1703CB, IC2 CP2102, U1 SP0504BAHTG, X1 TXC_7A

Commit message: Build settings, Eagle files
Other:
- note added: "Peter Antypas"
Changed lines of the file:
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@@
 <setting verticaltext="up"/>
 </settings>
-<grid distance="0.1" unitdist="inch" unit="inch" style="lines" multiple="1" display="no" altdistance="0.01" altunitdist="inch" altunit="inch"/>
+<grid distance="0.025" unitdist="inch" unit="inch" style="lines" multiple="1" display="no" altdistance="0.01" altunitdist="inch" altunit="inch"/>
 <layers>
 <layer number="1" name="Top" color="4" fill="1" visible="no" active="no"/>
@@
 <part name="PPS" library="adafruit" deviceset="PINHD-1X1" device=""/>
 <part name="GPS" library="adafruit" deviceset="PINHD-1X1" device=""/>
+<part name="FRAME1" library="SparkFun-Retired" deviceset="FRAME-A3" device=""/>
 </parts>
 <sheets>
 <sheet>
 <plain>
+<text x="138.43" y="-109.855" size="2.54" layer="94">Peter Antypas</text>
 </plain>
 <instances>
@@
 <attribute name="VALUE" x="-64.77" y="-73.025" size="1.778" layer="96" rot="R270"/>
 </instance>
+<instance part="FRAME1" gate="G$1" x="-190.5" y="-114.3"/>
 </instances>
 <busses>
