File: eagle/logic.brd (EAGLE design)
At the start: 73.6 x 36.8 mm, 76 parts, among them IC1 MCP1703CB, IC2 CP2102, U1 SP0504BAHTG, X1 TXC_7A

Commit message: More cleanup
Parts:
- added R10, R9: 10K, SparkFun-Passives:0603-RES
Connections:
- net +3V3: now also R10.2, R9.2
- net I2C_SCL: now also R9.1
- net I2C_SDA: now also R10.1
Routing:
- net +3V3: track 152.5 -> 157.5 mm
- net I2C_SDA: track 13.9 -> 14.6 mm
Other:
- board text added: "AIS Logic Stage Rev 3.2 (c) 2016 Peter Antypas"
- board text removed: "AIS Logic State Rev 3.1 (c) 2016 Peter Antypas"
Changed lines of the file:
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@@
 <layer number="27" name="tValues" color="7" fill="1" visible="yes" active="yes"/>
 <layer number="28" name="bValues" color="7" fill="1" visible="yes" active="yes"/>
-<layer number="29" name="tStop" color="7" fill="3" visible="no" active="yes"/>
-<layer number="30" name="bStop" color="7" fill="6" visible="no" active="yes"/>
+<layer number="29" name="tStop" color="7" fill="3" visible="yes" active="yes"/>
+<layer number="30" name="bStop" color="7" fill="6" visible="yes" active="yes"/>
 <layer number="31" name="tCream" color="7" fill="4" visible="no" active="yes"/>
 <layer number="32" name="bCream" color="7" fill="5" visible="no" active="yes"/>
@@
 <wire x1="73.6475" y1="36.82" x2="0" y2="36.82" width="0" layer="20"/>
 <wire x1="0" y1="36.82" x2="0" y2="0" width="0" layer="20"/>
-<rectangle x1="55.88" y1="22.225" x2="59.055" y2="25.4" layer="29"/>
+<rectangle x1="55.88" y1="22.225" x2="59.055" y2="25.4" layer="30"/>
 <text x="47.9425" y="21.2725" size="0.6096" layer="25" font="vector" ratio="10">5V</text>
 <text x="40.9575" y="21.2725" size="0.6096" layer="25" font="vector" ratio="10">GND</text>
@@
 <text x="73.3425" y="9.2075" size="0.6096" layer="25" font="vector" ratio="10" rot="R90">3V</text>
 <text x="53.0225" y="35.8775" size="0.6096" layer="25" font="vector" ratio="10">3V</text>
-<text x="44.7675" y="9.525" size="0.8128" layer="25" font="vector" ratio="10">AIS Logic State
-Rev 3.1
+<text x="44.7675" y="9.525" size="0.8128" layer="25" font="vector" ratio="10">AIS Logic Stage
+Rev 3.2
 (c) 2016 Peter Antypas</text>
+<rectangle x1="55.88" y1="22.225" x2="59.055" y2="25.4" layer="29"/>
 </plain>
 <attributes>
@@
 <attribute name="VALUE" x="6.985" y="5.3975" size="1.27" layer="27"/>
 </element>
+<element name="R9" library="SparkFun-Passives" package="0603-RES" value="10K" x="23.495" y="10.795"/>
+<element name="R10" library="SparkFun-Passives" package="0603-RES" value="10K" x="23.495" y="6.0325"/>
 </elements>
 <signals>
@@
 <via x="40.9575" y="29.5275" extent="1-16" drill="0.3302"/>
 <via x="22.86" y="18.0975" extent="1-16" drill="0.3302"/>
-<via x="25.0825" y="10.795" extent="1-16" drill="0.3302"/>
+<via x="24.765" y="8.255" extent="1-16" drill="0.3302"/>
 <via x="23.1775" y="13.97" extent="1-16" drill="0.3302"/>
 <via x="50.8" y="20.955" extent="1-16" drill="0.3302"/>
@@
 <wire x1="24.695" y1="7.305" x2="27.9425" y2="7.305" width="0.254" layer="1"/>
 <wire x1="27.9425" y1="7.305" x2="28.575" y2="7.9375" width="0.254" layer="1"/>
-<wire x1="28.575" y1="7.9375" x2="28.575" y2="12.28" width="0.254" layer="1"/>
+<wire x1="28.575" y1="7.9375" x2="28.575" y2="10.795" width="0.254" layer="1"/>
+<wire x1="28.575" y1="10.795" x2="28.575" y2="12.28" width="0.254" layer="1"/>
 <wire x1="28.575" y1="12.28" x2="28.4725" y2="12.3825" width="0.254" layer="1"/>
 <wire x1="53.2375" y1="20.955" x2="54.2925" y2="20.955" width="0.254" layer="1"/>
@@
 <wire x1="53.0225" y1="20.74" x2="53.2375" y2="20.955" width="0.254" layer="1"/>
 <wire x1="24.695" y1="7.305" x2="24.695" y2="6.3825" width="0.254" layer="1"/>
+<contactref element="R9" pad="2"/>
+<contactref element="R10" pad="2"/>
+<wire x1="24.345" y1="6.0325" x2="24.695" y2="6.0325" width="0.4064" layer="1"/>
+<wire x1="24.695" y1="6.0325" x2="24.695" y2="6.3825" width="0.4064" layer="1"/>
+<wire x1="24.345" y1="10.795" x2="28.575" y2="10.795" width="0.254" layer="1"/>
 </signal>
 <signal name="N$3">
@@
 <contactref element="U$1" pad="P$42"/>
 <contactref element="U$2" pad="1"/>
-<wire x1="22.295" y1="9.205" x2="22.295" y2="14.9925" width="0.254" layer="1"/>
+<wire x1="22.295" y1="9.205" x2="22.295" y2="10.4775" width="0.254" layer="1"/>
+<wire x1="22.295" y1="10.795" x2="22.295" y2="14.9925" width="0.254" layer="1"/>
 <wire x1="22.295" y1="14.9925" x2="23.495" y2="16.51" width="0.254" layer="1"/>
 <wire x1="23.495" y1="16.51" x2="26.5632375" y2="16.51" width="0.254" layer="1"/>
 <wire x1="26.5632375" y1="16.51" x2="27.29801875" y2="17.24478125" width="0.254" layer="1"/>
+<contactref element="R9" pad="1"/>
+<wire x1="22.645" y1="10.795" x2="22.295" y2="10.795" width="0.254" layer="1"/>
+<wire x1="22.295" y1="10.795" x2="22.295" y2="10.4775" width="0.254" layer="1"/>
 </signal>
 <signal name="I2C_SDA">
@@
 <wire x1="26.00034375" y1="15.24" x2="27.651571875" y2="16.891228125" width="0.254" layer="1"/>
 <wire x1="22.295" y1="7.305" x2="22.295" y2="6.3825" width="0.254" layer="1"/>
+<contactref element="R10" pad="1"/>
+<wire x1="22.645" y1="6.0325" x2="22.295" y2="6.0325" width="0.4064" layer="1"/>
+<wire x1="22.295" y1="6.0325" x2="22.295" y2="6.3825" width="0.4064" layer="1"/>
 </signal>
 <signal name="VDD1">

Commit message: Updated schematics with part values
Parts:
- C1, C2: value (none) -> 18pF
- C10, C9: value (none) -> 1uF
- C11, C12: value (none) -> DNP
- C3, C4, C5, C6, C7, C8: value (none) -> .1uF
- L1, L8: value (none) -> 0 ohm
- R1: value (none) -> 10k
- R2, R3, R4, R7, R8: value (none) -> 2.2k
Changed lines of the file:
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@@
 <?xml version="1.0" encoding="utf-8"?>
 <!DOCTYPE eagle SYSTEM "eagle.dtd">
-<eagle version="7.4.0">
+<eagle version="8.4.3">
 <drawing>
 <settings>
 <setting alwaysvectorfont="no"/>
+<setting keepoldvectorfont="yes"/>
 <setting verticaltext="up"/>
 </settings>
@@
 <param name="dpMaxLengthDifference" value="10mm"/>
 <param name="dpGapFactor" value="2.5"/>
-<param name="checkGrid" value="0"/>
 <param name="checkAngle" value="0"/>
 <param name="checkFont" value="1"/>
 <param name="checkRestrict" value="1"/>
+<param name="checkStop" value="0"/>
 <param name="useDiameter" value="13"/>
 <param name="maxErrors" value="50"/>
@@
 <attribute name="VALUE" x="19.685" y="33.655" size="1.27" layer="27" rot="R90"/>
 </element>
-<element name="C1" library="SparkFun-Capacitors" package="0603-CAP" value="" x="39.0525" y="11.43" rot="R270"/>
-<element name="C10" library="SparkFun-Capacitors" package="0805" value="" x="58.42" y="19.3675" rot="R180"/>
-<element name="C11" library="SparkFun-Capacitors" package="0603-CAP" value="" x="52.3875" y="20.955" rot="R180"/>
-<element name="C12" library="SparkFun-Capacitors" package="0603-CAP" value="" x="58.1025" y="13.97"/>
+<element name="C1" library="SparkFun-Capacitors" package="0603-CAP" value="18pF" x="39.0525" y="11.43" rot="R270"/>
+<element name="C10" library="SparkFun-Capacitors" package="0805" value="1uF" x="58.42" y="19.3675" rot="R180"/>
+<element name="C11" library="SparkFun-Capacitors" package="0603-CAP" value="DNP" x="52.3875" y="20.955" rot="R180"/>
+<element name="C12" library="SparkFun-Capacitors" package="0603-CAP" value="DNP" x="58.1025" y="13.97"/>
 <element name="C13" library="SparkFun-Capacitors" package="0603-CAP" value="1nF" x="5.715" y="29.5275" rot="R180"/>
 <element name="C14" library="SparkFun-Capacitors" package="0603-CAP" value="1uF" x="5.715" y="28.2575" rot="R180"/>
-<element name="C2" library="SparkFun-Capacitors" package="0603-CAP" value="" x="31.4325" y="11.43" rot="R90"/>
-<element name="C3" library="SparkFun-Capacitors" package="0603-CAP" value="" x="33.655" y="27.6225"/>
-<element name="C4" library="SparkFun-Capacitors" package="0603-CAP" value="" x="27.6225" y="12.3825" rot="R180"/>
-<element name="C5" library="SparkFun-Capacitors" package="0603-CAP" value="" x="23.8125" y="20.955" rot="R90"/>
-<element name="C6" library="SparkFun-Capacitors" package="0603-CAP" value="" x="30.7975" y="27.6225" rot="R180"/>
-<element name="C7" library="SparkFun-Capacitors" package="0603-CAP" value="" x="13.6525" y="3.4925" rot="R270"/>
-<element name="C8" library="SparkFun-Capacitors" package="0603-CAP" value="" x="6.6675" y="34.29" smashed="yes" rot="R90">
+<element name="C2" library="SparkFun-Capacitors" package="0603-CAP" value="18pF" x="31.4325" y="11.43" rot="R90"/>
+<element name="C3" library="SparkFun-Capacitors" package="0603-CAP" value=".1uF" x="33.655" y="27.6225"/>
+<element name="C4" library="SparkFun-Capacitors" package="0603-CAP" value=".1uF" x="27.6225" y="12.3825" rot="R180"/>
+<element name="C5" library="SparkFun-Capacitors" package="0603-CAP" value=".1uF" x="23.8125" y="20.955" rot="R90"/>
+<element name="C6" library="SparkFun-Capacitors" package="0603-CAP" value=".1uF" x="30.7975" y="27.6225" rot="R180"/>
+<element name="C7" library="SparkFun-Capacitors" package="0603-CAP" value=".1uF" x="13.6525" y="3.4925" rot="R270"/>
+<element name="C8" library="SparkFun-Capacitors" package="0603-CAP" value=".1uF" x="6.6675" y="34.29" smashed="yes" rot="R90">
 <attribute name="NAME" x="5.9055" y="33.401" size="0.4064" layer="25" font="vector" rot="R90"/>
 <attribute name="VALUE" x="7.8105" y="33.274" size="0.4064" layer="27" font="vector" rot="R90"/>
 </element>
-<element name="C9" library="SparkFun-Capacitors" package="0805" value="" x="58.1025" y="12.7"/>
+<element name="C9" library="SparkFun-Capacitors" package="0805" value="1uF" x="58.1025" y="12.7"/>
 <element name="CLK1" library="adafruit" package="1X01" value="" x="63.8175" y="34.29" smashed="yes">
 <attribute name="NAME" x="62.7888" y="35.8013" size="0.6096" layer="25" font="vector" ratio="10"/>
@@
 <element name="IC1" library="linear" package="SOT23" value="MCP1703CB" x="58.42" y="16.8275" smashed="yes" rot="R90"/>
 <element name="IC2" library="silabs" package="MLP28" value="CP2102" x="57.4675" y="23.8125" smashed="yes" rot="MR0">
-<attribute name="OC_NEWARK" value="30K5635" x="57.4675" y="23.8125" size="1.778" layer="28" rot="MR0" display="off"/>
 <attribute name="MF" value="FARNELL" x="57.4675" y="23.8125" size="1.778" layer="28" rot="MR0" display="off"/>
-<attribute name="OC_FARNELL" value="9282130" x="57.4675" y="23.8125" size="1.778" layer="28" rot="MR0" display="off"/>
 <attribute name="MPN" value="CP2102-GM" x="57.4675" y="23.8125" size="1.778" layer="28" rot="MR0" display="off"/>
 <attribute name="NAME" x="60.0075" y="26.9875" size="1.27" layer="26" rot="MR0"/>
-</element>
-<element name="L1" library="SparkFun-Passives" package="0603" value="" x="58.42" y="20.6375" smashed="yes" rot="R180">
+<attribute name="OC_FARNELL" value="9282130" x="57.4675" y="23.8125" size="1.778" layer="28" rot="MR0" display="off"/>
+<attribute name="OC_NEWARK" value="30K5635" x="57.4675" y="23.8125" size="1.778" layer="28" rot="MR0" display="off"/>
+</element>
+<element name="L1" library="SparkFun-Passives" package="0603" value="0 ohm" x="58.42" y="20.6375" smashed="yes" rot="R180">
+<attribute name="NAME" x="59.309" y="19.8755" size="0.4064" layer="25" font="vector" rot="R180"/>
 <attribute name="PROD_ID" value="RES-07859" x="58.42" y="20.6375" size="1.778" layer="27" rot="R180" display="off"/>
-<attribute name="NAME" x="59.309" y="19.8755" size="0.4064" layer="25" font="vector" rot="R180"/>
 <attribute name="VALUE" x="59.436" y="21.7805" size="0.4064" layer="27" font="vector" rot="R180"/>
 </element>
-<element name="L8" library="SparkFun-Passives" package="0603" value="" x="6.6675" y="31.4325" rot="R270"/>
+<element name="L8" library="SparkFun-Passives" package="0603" value="0 ohm" x="6.6675" y="31.4325" rot="R270"/>
 <element name="GRN" library="adafruit" package="CHIP-LED0603" value="" x="21.59" y="34.29" smashed="yes">
 <attribute name="NAME" x="22.5425" y="36.5125" size="0.6096" layer="25" font="vector" ratio="10" rot="R180"/>
@@
 <attribute name="VALUE" x="57.4675" y="-0.635" size="1.27" layer="27"/>
 </element>
-<element name="R1" library="SparkFun-Passives" package="0603-RES" value="" x="24.4475" y="13.97"/>
-<element name="R2" library="SparkFun-Passives" package="0603-RES" value="" x="23.495" y="31.75" rot="R270"/>
-<element name="R3" library="SparkFun-Passives" package="0603-RES" value="" x="19.685" y="31.75" rot="R270"/>
-<element name="R4" library="SparkFun-Passives" package="0603-RES" value="" x="17.78" y="31.75" rot="R270"/>
+<element name="R1" library="SparkFun-Passives" package="0603-RES" value="10k" x="24.4475" y="13.97"/>
+<element name="R2" library="SparkFun-Passives" package="0603-RES" value="2.2k" x="23.495" y="31.75" rot="R270"/>
+<element name="R3" library="SparkFun-Passives" package="0603-RES" value="2.2k" x="19.685" y="31.75" rot="R270"/>
+<element name="R4" library="SparkFun-Passives" package="0603-RES" value="2.2k" x="17.78" y="31.75" rot="R270"/>
 <element name="R5" library="SparkFun-Passives" package="0603-RES" value="4K7" x="59.3725" y="19.3675" rot="MR0"/>
 <element name="R6" library="SparkFun-Passives" package="0603-RES" value="10K" x="56.1975" y="19.3675" rot="MR180"/>
-<element name="R7" library="SparkFun-Passives" package="0603-RES" value="" x="21.59" y="31.75" rot="R270"/>
-<element name="R8" library="SparkFun-Passives" package="0603-RES" value="" x="9.8425" y="31.4325" rot="R270"/>
+<element name="R7" library="SparkFun-Passives" package="0603-RES" value="2.2k" x="21.59" y="31.75" rot="R270"/>
+<element name="R8" library="SparkFun-Passives" package="0603-RES" value="2.2k" x="9.8425" y="31.4325" rot="R270"/>
 <element name="RED" library="adafruit" package="CHIP-LED0603" value="" x="23.495" y="34.29" smashed="yes">
 <attribute name="NAME" x="24.765" y="36.5125" size="0.6096" layer="25" font="vector" ratio="10" rot="R180"/>
@@
 <element name="U$3" library="GeekAmmo" package="7914G" value="TACTILE-SWITCH-7914G" x="11.7475" y="2.2225" smashed="yes" rot="R90"/>
 <element name="U1" library="Littelfuse_By_element14_Batch_1" package="SOT95P280X145-5N" value="SP0504BAHTG" x="61.9125" y="20.955" smashed="yes" rot="R90">
+<attribute name="MPN" value="SP0504BAHTG" x="61.9125" y="20.955" size="1.778" layer="27" rot="R90" display="off"/>
+<attribute name="OC_FARNELL" value="1827634" x="61.9125" y="20.955" size="1.778" layer="27" rot="R90" display="off"/>
 <attribute name="OC_NEWARK" value="92K8961" x="61.9125" y="20.955" size="1.778" layer="27" rot="R90" display="off"/>
 <attribute name="PACKAGE" value="SOT-23-3" x="61.9125" y="20.955" size="1.778" layer="27" rot="R90" display="off"/>
 <attribute name="SUPPLIER" value="LITTELFUSE" x="61.9125" y="20.955" size="1.778" layer="27" rot="R90" display="off"/>
-<attribute name="OC_FARNELL" value="1827634" x="61.9125" y="20.955" size="1.778" layer="27" rot="R90" display="off"/>
-<attribute name="MPN" value="SP0504BAHTG" x="61.9125" y="20.955" size="1.778" layer="27" rot="R90" display="off"/>
 </element>
 <element name="U2" library="adafruit" package="FGPMMOPA6H" value="" x="9.525" y="18.415" smashed="yes">
