File: eagle/logic.sch (EAGLE design)
At the start: 76 parts, among them IC1 MCP1703CB, IC2 CP2102, U1 SP0504BAHTG, X1 TXC_7A

Commit message: More cleanup
Parts:
- added R10, R9: 10K, SparkFun-Passives:RESISTOR0603-RES
Connections:
- net +3V3: now also R10.2, R9.2
- net I2C_SCL: now also R9.1
- net I2C_SDA: now also R10.1
Changed lines of the file:
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@@
 <part name="GPS" library="adafruit" deviceset="PINHD-1X1" device=""/>
 <part name="FRAME1" library="SparkFun-Retired" deviceset="FRAME-A3" device=""/>
+<part name="R9" library="SparkFun-Passives" deviceset="RESISTOR" device="0603-RES" value="10K"/>
+<part name="R10" library="SparkFun-Passives" deviceset="RESISTOR" device="0603-RES" value="10K"/>
+<part name="+3V7" library="supply1" deviceset="+3V3" device=""/>
 </parts>
 <sheets>
@@
 </instance>
 <instance part="FRAME1" gate="G$1" x="-190.5" y="-114.3"/>
+<instance part="R9" gate="G$1" x="-67.31" y="-10.16" rot="R90"/>
+<instance part="R10" gate="G$1" x="-71.12" y="-25.4" rot="R90"/>
+<instance part="+3V7" gate="G$1" x="-67.31" y="0" smashed="yes">
+<attribute name="VALUE" x="-63.5" y="3.81" size="1.778" layer="96" rot="R180"/>
+</instance>
 </instances>
 <busses>
@@
 <pinref part="+3V6" gate="G$1" pin="+3V3"/>
 </segment>
+<segment>
+<pinref part="R10" gate="G$1" pin="2"/>
+<wire x1="-71.12" y1="-20.32" x2="-71.12" y2="-5.08" width="0.1524" layer="91"/>
+<pinref part="R9" gate="G$1" pin="2"/>
+<wire x1="-71.12" y1="-5.08" x2="-67.31" y2="-5.08" width="0.1524" layer="91"/>
+<wire x1="-67.31" y1="-5.08" x2="-67.31" y2="-2.54" width="0.1524" layer="91"/>
+<junction x="-67.31" y="-5.08"/>
+<pinref part="+3V7" gate="G$1" pin="+3V3"/>
+</segment>
 </net>
 <net name="N$3" class="0">
@@
 <segment>
 <pinref part="U$2" gate="G$1" pin="SCL"/>
-<wire x1="-60.96" y1="-15.24" x2="-73.66" y2="-15.24" width="0.1524" layer="91"/>
+<wire x1="-60.96" y1="-15.24" x2="-67.31" y2="-15.24" width="0.1524" layer="91"/>
 <label x="-74.93" y="-15.24" size="1.778" layer="95" rot="R180" xref="yes"/>
+<pinref part="R9" gate="G$1" pin="1"/>
+<wire x1="-67.31" y1="-15.24" x2="-73.66" y2="-15.24" width="0.1524" layer="91"/>
+<junction x="-67.31" y="-15.24"/>
 </segment>
 </net>
@@
 <pinref part="U$2" gate="G$1" pin="SDA"/>
 <label x="-75.565" y="-30.48" size="1.778" layer="95" rot="R180" xref="yes"/>
-<wire x1="-60.96" y1="-30.48" x2="-74.93" y2="-30.48" width="0.1524" layer="91"/>
-</segment>
-</net>
+<wire x1="-60.96" y1="-30.48" x2="-71.12" y2="-30.48" width="0.1524" layer="91"/>
+<pinref part="R10" gate="G$1" pin="1"/>
+<wire x1="-71.12" y1="-30.48" x2="-74.93" y2="-30.48" width="0.1524" layer="91"/>
+<junction x="-71.12" y="-30.48"/>
+</segment>
+</net>

Commit message: Updated schematics with part values
Parts:
- C1, C2: value (none) -> 18pF
- C10, C9: value (none) -> 1uF
- C11, C12: value (none) -> DNP
- C3, C4, C5, C6, C7, C8: value (none) -> .1uF
- L1, L8: value (none) -> 0 ohm
- R1: value (none) -> 10k
- R2, R3, R4, R7, R8: value (none) -> 2.2k
Other:
- moved on the sheet: C10, C12, IC1
