File: latest/CAD/Board-6.2/transponder-6.2.0.brd (EAGLE design)
At the start: 90 x 25.4 mm, 126 parts, among them U1 AP3211KTR-G1, U10 1575AT43A0040E, U11 SI4463, U12 SI4463, U13 STM32L412KBU6, U15 SKY13330-397LF, U3 LDFPUR, U4 DMN63D8LDW-7, U5 LP5907QMFX-1.8Q1, U6 24LC01B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

Commit message: Checkpoint
Parts:
- removed TX_OFF: TPTP12R, testpad:TP12R
- moved GND2 13.5 mm to (22.2, 6.00)
- moved SWDIO 3.00 mm to (17.0, 4.00)
- moved SWCLK 2.00 mm to (19.0, 4.00)
- moved V_IN 1.80 mm to (16.1, 19.0)
- moved NRST 1.00 mm to (21.0, 4.00)
- moved C12 0.50 mm to (17.3, 6.90)
- moved C5 0.40 mm to (18.8, 7.00)
- moved D2 0.40 mm to (6.40, 22.5)
- moved C6 0.30 mm to (20.5, 17.0)
- moved L10 0.22 mm to (79.9, 19.4)
- moved C44 0.20 mm to (77.4, 15.8)
- moved C1 0.20 mm to (20.4, 7.00)
- moved C30 0.14 mm to (63.9, 19.2)
- moved C23 0.10 mm to (50.9, 20.7)
- moved C24 0.10 mm to (54.7, 20.7)
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Connections:
- net TX_DISABLE: no longer TX_OFF.TP
Routing:
- net TX_DISABLE: track 21.3 -> 18.0 mm, vias 2 -> 1
- net V_IN: track 16.0 -> 17.4 mm
- net SWCLK: track 18.1 -> 19.0 mm
- net NRST: track 24.7 -> 24.0 mm
Other:
- outline, holes or cut-outs redrawn
