File: latest/CAD/Board-6.2/transponder-6.2.0.sch (EAGLE design)
At the start: 126 parts, among them U1 AP3211KTR-G1, U10 1575AT43A0040E, U11 SI4463, U12 SI4463, U13 STM32L412KBU6, U15 SKY13330-397LF, U3 LDFPUR, U4 DMN63D8LDW-7, U5 LP5907QMFX-1.8Q1, U6 24LC01B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

Commit message: Checkpoint
Parts:
- removed TX_OFF: TPTP12R, testpad:TPTP12R
Connections:
- net TX_DISABLE: no longer TX_OFF.TP
Changed lines of the file:
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@@
 <part name="SUPPLY40" library="supply2" deviceset="GND" device=""/>
 <part name="SUPPLY61" library="supply2" deviceset="GND" device=""/>
-<part name="TX_OFF" library="testpad" deviceset="TP" device="TP12R" value="TPTP12R">
-<attribute name="DNP" value="T"/>
-</part>
 <part name="U4" library="diodesinc" deviceset="DMN63D8LDW" device="" value="DMN63D8LDW-7">
 <attribute name="PARTNO" value="DMN63D8LDW-7"/>
@@
 </instance>
 <instance part="SUPPLY16" gate="GND" x="104.14" y="25.4" smashed="yes"/>
-<instance part="TX_OFF" gate="G$1" x="152.4" y="114.3" smashed="yes">
-<attribute name="NAME" x="151.13" y="115.57" size="1.27" layer="95"/>
-<attribute name="TP_SIGNAL_NAME" x="153.67" y="113.03" size="1.778" layer="97"/>
-<attribute name="DNP" x="152.4" y="114.3" size="1.27" layer="96" display="off"/>
-</instance>
 </instances>
 <busses>
@@
 <segment>
 <pinref part="U13" gate="G$1" pin="PA12"/>
-<wire x1="147.32" y1="111.76" x2="152.4" y2="111.76" width="0.1524" layer="91"/>
 <label x="160.02" y="111.76" size="1.27" layer="95" xref="yes"/>
-<pinref part="TX_OFF" gate="G$1" pin="TP"/>
-<wire x1="152.4" y1="111.76" x2="160.02" y2="111.76" width="0.1524" layer="91"/>
-<junction x="152.4" y="111.76"/>
-</segment>
-</net>
+<wire x1="147.32" y1="111.76" x2="160.02" y2="111.76" width="0.1524" layer="91"/>
+</segment>
+</net>
