File: latest/CAD/Board-7.0/transponder-7.0.0.brd (EAGLE design)
At the start: 90 x 25.4 mm, 130 parts, among them Q1 DMP3099L-7, Q2 DMP3099L-7, U1 AP63203WU-7, U10 1575AT43A0040E, U11 SI4463, U12 SI4463, U13 STM32L412K8U6, U15 SKY13330-397LF, U2 PSA4-5043+, U3 LDFPUR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

Commit message: 7.x assembly variants
Parts:
- R2, R3, R7: value 1k -> 1k1
- renumbered U$6 to U16
Changed lines of the file:
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@@
 </attributes>
 <variantdefs>
+<variantdef name="Supercap"/>
+<variantdef name="No supercap"/>
 </variantdefs>
 <classes>
@@
 <element name="C37" library="MyPassives" package="0603" value="47pF" x="73.6" y="21.1" smashed="yes" rot="R90">
 <attribute name="NAME" x="73.6745" y="22.938" size="0.6096" layer="25" font="vector" rot="R90"/>
-<attribute name="PARTNO" value="Murata Electronics" x="73.6" y="21.1" size="1.778" layer="27" rot="R90" display="off"/>
+<attribute name="PARTNO" value="GRM1885C1H470JA01J" x="73.6" y="21.1" size="1.778" layer="27" rot="R90" display="off"/>
 <attribute name="VALUE" x="74.997" y="20.084" size="0.6096" layer="27" font="vector" rot="R90"/>
 </element>
@@
 <attribute name="PRICE" value="None" x="73.1" y="10.4" size="1.778" layer="27" rot="R270" display="off"/>
 </element>
-<element name="U$6" library="rfmi" package="SAW_FILTER1" value="SF2147D" x="58.8" y="11" smashed="yes" rot="R180">
+<element name="U16" library="rfmi" package="SAW_FILTER1" value="SF2147D" x="58.8" y="11" smashed="yes" rot="R180">
 <attribute name="NAME" x="60.1" y="8.3" size="0.6096" layer="25" font="vector" rot="R180"/>
 <attribute name="PARTNO" value="SF2147D" x="58.8" y="11" size="1.778" layer="27" rot="R180" display="off"/>
@@
 <attribute name="PARTNO" value="RC0603FR-070RL" x="26.3" y="23.6" size="1.778" layer="27" display="off"/>
 </element>
-<element name="R2" library="MyPassives" package="0603" value="1k" x="22.7" y="9.9" smashed="yes" rot="R90">
+<element name="R2" library="MyPassives" package="0603" value="1k1" x="22.7" y="9.9" smashed="yes" rot="R90">
 <attribute name="NAME" x="22" y="8.5" size="0.6096" layer="25" font="vector" rot="R90"/>
-<attribute name="PARTNO" value="RC0603JR-071KL" x="22.7" y="9.9" size="1.778" layer="27" rot="R90" display="off"/>
-</element>
-<element name="R3" library="MyPassives" package="0603" value="1k" x="27.8" y="17.8" smashed="yes" rot="R180">
+<attribute name="PARTNO" value="RC0603JR-071K1L" x="22.7" y="9.9" size="1.778" layer="27" rot="R90" display="off"/>
+</element>
+<element name="R3" library="MyPassives" package="0603" value="1k1" x="27.8" y="17.8" smashed="yes" rot="R180">
 <attribute name="NAME" x="29.2" y="17.1" size="0.6096" layer="25" font="vector" rot="R180"/>
-<attribute name="PARTNO" value="RC0603JR-071KL" x="27.8" y="17.8" size="1.778" layer="27" rot="R180" display="off"/>
-</element>
-<element name="R7" library="MyPassives" package="0603" value="1k" x="23.2" y="18.3" smashed="yes" rot="R90">
+<attribute name="PARTNO" value="RC0603JR-071K1L" x="27.8" y="17.8" size="1.778" layer="27" rot="R180" display="off"/>
+</element>
+<element name="R7" library="MyPassives" package="0603" value="1k1" x="23.2" y="18.3" smashed="yes" rot="R90">
 <attribute name="NAME" x="22.5" y="16.9" size="0.6096" layer="25" font="vector" rot="R90"/>
-<attribute name="PARTNO" value="RC0603JR-071KL" x="23.2" y="18.3" size="1.778" layer="27" rot="R90" display="off"/>
+<attribute name="PARTNO" value="RC0603JR-071K1L" x="23.2" y="18.3" size="1.778" layer="27" rot="R90" display="off"/>
 </element>
 </elements>
@@
 <contactref element="U2" pad="4"/>
 <contactref element="U2" pad="2"/>
-<contactref element="U$6" pad="P$4"/>
-<contactref element="U$6" pad="P$3"/>
-<contactref element="U$6" pad="P$6"/>
-<contactref element="U$6" pad="P$1"/>
+<contactref element="U16" pad="P$4"/>
+<contactref element="U16" pad="P$3"/>
+<contactref element="U16" pad="P$6"/>
+<contactref element="U16" pad="P$1"/>
 <contactref element="C10" pad="P$1"/>
 <via x="75.5" y="9.2" extent="1-16" drill="0.254"/>
@@
 </signal>
 <signal name="N$4">
-<contactref element="U$6" pad="P$2"/>
+<contactref element="U16" pad="P$2"/>
 <contactref element="L14" pad="P$1"/>
 <wire x1="61.7" y1="11" x2="60.3" y2="11" width="1" layer="1"/>
@@
 </signal>
 <signal name="N$33">
-<contactref element="U$6" pad="P$5"/>
+<contactref element="U16" pad="P$5"/>
 <contactref element="L16" pad="P$2"/>
 <wire x1="57.2" y1="11" x2="55.9" y2="11" width="1" layer="1"/>
