File: latest/CAD/NMEA0183Breakout/NMEA0183Breakout-3.0.brd (EAGLE design)
At the start: 52 x 42 mm, 35 parts, among them IC1 LD2985BM50R, J1 10118194-0001LF, J2 RJ-82A86MMNL, Q1 DMP3099L-7, Q2 DMP3099L-7, Q3 DMP3099L-7, Q4 BSS138, U1 DS8921M

Commit message: Updated CAD
Parts:
- added C6: 1uF, MyPassives:0603
- moved C1 24.4 mm to (19.3, 17.5), turned to 270 degrees
- moved IC1 21.2 mm to (16.5, 17.4), turned to 270 degrees
- moved R9 20.6 mm to (45.3, 18.8), turned to 90 degrees
- moved Q2 18.3 mm to (29.5, 18.0), turned to 0 degrees
- moved C2 18.1 mm to (13.4, 17.2), turned to 90 degrees
- moved R5 11.9 mm to (30.2, 20.8), turned to 0 degrees
- moved R6 5.30 mm to (33.9, 10.9), turned to 270 degrees
- moved R7 2.52 mm to (31.9, 10.9), turned to 270 degrees
Connections:
- new net N$5: R9.P$2, S2.P$2
- net GND: now also C6.P$2; no longer R9.P$1
- net TX_DISABLE: now also C6.P$1, R9.P$1; no longer R9.P$2, S2.P$2
Routing:
- net 5V: track 83.2 -> 65.6 mm, vias 3 -> 2
- net TX_DISABLE: track 31.5 -> 45.0 mm, vias 0 -> 2
- net V_OUT: track 40.4 -> 51.2 mm
- net N$5: track 0.00 -> 9.97 mm
- net AIS_TX_EVENT: track 19.6 -> 29.5 mm, vias 2 -> 3
- net S2: track 15.9 -> 20.8 mm
- net TRANSPONDER_UART_RX: track 38.6 -> 34.3 mm, vias 2 -> 0
- net S1: track 21.6 -> 20.4 mm
- net N$6: track 2.60 -> 1.74 mm
Other:
- outline, holes or cut-outs redrawn
- board text added: "MAIANA Universal Breakout Rev3.0 (NMEA0183+USB) (c)2021 P. Antypas"
- board text removed: "MAIANA Universal Breakout Rev 2.0 (UART+0183+USB) (c)2021 P. Antypas"
