File: latest/CAD/USBBreakout/USBBreakout-2.0.brd (EAGLE design)
At the start: 36 x 46 mm, 31 parts, among them IC1 MIC5203-3.3YM5-TR, J1 OSTVN02A150, J2 10118194-0001LF, J3 RJ-82A86MMNL, Q1 DMP3099L-7, Q2 DMP3099L-7, Q3 DMP3099L-7, Q4 BSS138

Commit message: Updated CAD
Parts:
- added C3: 1uF, MyPassives:0603
- moved R6 5.92 mm to (28.5, 17.7), turned to 90 degrees
Connections:
- new net N$5: R6.P$1, SILENT.2
- net GND: now also C3.P$2; no longer R6.P$2
- net TX_DISABLE: now also C3.P$1, R6.P$2; no longer R6.P$1, SILENT.2
Routing:
- net N$5: track 0.00 -> 3.92 mm
- net TX_DISABLE: track 59.2 -> 55.9 mm
Other:
- board text added: "MAIANA USBControl Box Rev 2.0"
- board text removed: "MAIANA Control Box Rev 1.3"
Changed lines of the file:
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@@
 <text x="7.5" y="40.8" size="2.54" layer="26" font="vector" rot="MR0">+</text>
 <text x="10.2" y="40.9" size="2.54" layer="26" font="vector" rot="MR0">-</text>
-<text x="34.8" y="16.8" size="0.8128" layer="25" font="vector" rot="R90">MAIANA Control Box
-Rev 1.3</text>
+<text x="34.8" y="16.8" size="0.8128" layer="25" font="vector" rot="R90">MAIANA USBControl Box
+Rev 2.0</text>
 </plain>
 <attributes>
@@
 <attribute name="VALUE" x="31.8" y="31.9" size="0.6096" layer="27" font="vector" rot="R270"/>
 </element>
-<element name="R6" library="MyPassives" package="0603" value="10k" x="32.1" y="13" smashed="yes" rot="R270">
-<attribute name="NAME" x="32.8" y="14.4" size="0.6096" layer="25" font="vector" rot="R270"/>
-<attribute name="PARTNO" value="" x="32.1" y="13" size="1.778" layer="27" font="vector" rot="R270" display="off"/>
-<attribute name="VALUE" x="32" y="13.6" size="0.6096" layer="27" font="vector" rot="R270"/>
+<element name="R6" library="MyPassives" package="0603" value="10k" x="28.5" y="17.7" smashed="yes" rot="R90">
+<attribute name="NAME" x="28.6" y="19.4" size="0.6096" layer="25" font="vector" rot="R90"/>
+<attribute name="PARTNO" value="" x="28.5" y="17.7" size="1.778" layer="27" rot="R90" display="off"/>
+<attribute name="VALUE" x="28.8" y="17.1" size="0.6096" layer="27" font="vector" rot="R90"/>
+</element>
+<element name="C3" library="MyPassives" package="0603" value="1uF" x="30.5" y="17.7" smashed="yes" rot="R270">
+<attribute name="NAME" x="30.8" y="19.4" size="0.6096" layer="25" font="vector" rot="R90"/>
+<attribute name="PARTNO" value="" x="30.5" y="17.7" size="1.778" layer="27" rot="R270" display="off"/>
+<attribute name="VALUE" x="30.2" y="18.3" size="0.6096" layer="27" font="vector" rot="R270"/>
 </element>
 </elements>
@@
 <contactref element="ON_OFF" pad="1"/>
 <contactref element="R7" pad="P$2"/>
-<contactref element="R6" pad="P$2"/>
 <polygon width="0.1524" layer="1">
 <vertex x="-1" y="47"/>
@@
 <contactref element="J2" pad="5"/>
 <contactref element="SILENT" pad="3"/>
+<contactref element="C3" pad="P$2"/>
 </signal>
 <signal name="TRANSPONDER_UART_TX">
@@
 <wire x1="7.5714" y1="15.5786" x2="8.5" y2="14.65" width="0.1524" layer="1"/>
 <wire x1="18.4" y1="27" x2="12.1" y2="20.7" width="0.1524" layer="16"/>
-<contactref element="SILENT" pad="2"/>
-<contactref element="R6" pad="P$1"/>
-<wire x1="31.15" y1="14.75" x2="32.1" y2="13.8" width="0.1524" layer="1"/>
-<wire x1="26" y1="14.75" x2="26.1" y2="14.75" width="0.1524" layer="1"/>
-<wire x1="26.1" y1="14.75" x2="31.15" y2="14.75" width="0.1524" layer="1"/>
 <wire x1="24.75" y1="31.5" x2="25.5" y2="30.75" width="0.1524" layer="1"/>
 <wire x1="25.5" y1="30.75" x2="25.5" y2="30.5" width="0.1524" layer="1"/>
@@
 <wire x1="26" y1="18.2" x2="26" y2="16.8" width="0.1524" layer="16"/>
 <via x="26" y="16.8" extent="1-16" drill="0.3"/>
-<wire x1="26" y1="16.8" x2="26" y2="14.85" width="0.1524" layer="1"/>
-<wire x1="26" y1="14.85" x2="26.1" y2="14.75" width="0.1524" layer="1"/>
+<contactref element="R6" pad="P$2"/>
+<contactref element="C3" pad="P$1"/>
+<wire x1="28.5" y1="18.5" x2="30.5" y2="18.5" width="0.1524" layer="1"/>
+<wire x1="26" y1="16.8" x2="27.7" y2="18.5" width="0.1524" layer="1"/>
+<wire x1="27.7" y1="18.5" x2="28.5" y2="18.5" width="0.1524" layer="1"/>
 </signal>
 <signal name="GPS_STATUS">
@@
 <wire x1="18.8" y1="28.8" x2="17.6" y2="28.8" width="0.1524" layer="1"/>
 </signal>
+<signal name="N$5">
+<contactref element="SILENT" pad="2"/>
+<contactref element="R6" pad="P$1"/>
+<wire x1="28.5" y1="16.9" x2="28.5" y2="16" width="0.1524" layer="1"/>
+<wire x1="28.5" y1="16" x2="27.25" y2="14.75" width="0.1524" layer="1"/>
+<wire x1="27.25" y1="14.75" x2="26" y2="14.75" width="0.1524" layer="1"/>
+</signal>
 </signals>
